Commit message: state estimation runs (terribly)

File: urdf/autonav_bot.urdf (robot description, URDF)
Before this commit: robot my_robot, 3 links, 2 joints
Links:
- removed link camera_link
- removed link imu_link
- added link camera; visual box size=0.02 0.06 0.02
- added link imu; visual box size=0.04 0.03 0.02
Joints:
- joint base_to_camera_joint: child camera_link -> camera
- joint base_to_imu_joint: child imu_link -> imu; origin xyz=0 0 -.01 rpy=0 0 0 -> xyz=0 0 0 rpy=0 0 0

Commit message: mod urdf and launch file TFs

File: urdf/autonav_bot.urdf (robot description, URDF)
Before this commit: robot my_robot, 3 links, 2 joints
Links:
- removed link camera_link
- removed link imu_link
- added link camera; visual box size=0.02 0.06 0.02
- added link imu; visual box size=0.04 0.03 0.02
Joints:
- joint base_to_camera_joint: child camera_link -> camera
- joint base_to_imu_joint: child imu_link -> imu

Commit message: gmapping fixes - it runs kinda

File: urdf/autonav_bot.urdf (robot description, URDF)
Before this commit: robot my_robot, 3 links, 2 joints
Joints:
- joint base_to_imu_joint: origin xyz=0 0 0 rpy=0 0 0 -> xyz=0 0 -0.01 rpy=0 0 0
